File: BJTCC-12V/bjtcc.sch (KiCad schematic (older format))
At the start: 9 parts, among them J1 Screw_Terminal_1x04, P1 CONN_02X01, Q1 ASZ15, Q2 ASZ15

Commit message: rough placing footprints on PCB
Parts:
- Q1, Q2: footprint TO_SOT_Packages_THT:TO-247_PadsOnly_Neutral123 -> TO_SOT_Packages_THT:TO3
Changed lines of the file:
@@
 F 0 "Q1" H 3700 3850 50  0000 L CNN
 F 1 "ASZ15" H 3600 4200 50  0000 L CNN
-F 2 "TO_SOT_Packages_THT:TO-247_PadsOnly_Neutral123" H 4000 4100 50  0001 C CNN
+F 2 "TO_SOT_Packages_THT:TO3" H 4000 4100 50  0001 C CNN
 F 3 "" H 3800 4000 50  0000 C CNN
 	1    3800 4000
@@
 F 0 "Q2" H 4100 3850 50  0000 L CNN
 F 1 "ASZ15" H 4000 4200 50  0000 L CNN
-F 2 "TO_SOT_Packages_THT:TO-247_PadsOnly_Neutral123" H 4400 4100 50  0001 C CNN
+F 2 "TO_SOT_Packages_THT:TO3" H 4400 4100 50  0001 C CNN
 F 3 "" H 4200 4000 50  0000 C CNN
 	1    4200 4000
