File: BJTSICC-3V/kicad/pcb/bjtcc.sch (KiCad schematic (older format))
At the start: 9 parts, among them J1 Screw_Terminal_1x04, P1 CONN_02X01, Q1 ASZ15, Q2 ASZ15

Commit message: BJT version with Si and Ge
Parts:
- removed Q1, Q2: ASZ15, TO_SOT_Packages_THT:TO3, symbol Q_PNP_BCE
- added Q1, Q2: KD503, symbol Q_NPN_BCE
- R1: value 47 -> 33
- R2: renamed from R3; value 47 -> 33
- renumbered R2 to R3
Other:
- note added: "R1,R2: 15..100 ohm"
Changed lines of the file:
@@
 $EndDescr
-$Comp
-L Q_PNP_BCE Q1
-U 1 1 5911CAA3
-P 3800 4000
-F 0 "Q1" H 3700 3850 50  0000 L CNN
-F 1 "ASZ15" H 3600 4200 50  0000 L CNN
-F 2 "TO_SOT_Packages_THT:TO3" H 4000 4100 50  0001 C CNN
-F 3 "" H 3800 4000 50  0000 C CNN
-	1    3800 4000
-	1    0    0    1
-$EndComp
 $Comp
 L D_Schottky D1
@@
 F 3 "" H 3350 4000 50  0000 C CNN
 	1    3350 4000
-	1    0    0    -1
+	-1   0    0    1
 $EndComp
 $Comp
@@
 P 3450 3700
 F 0 "R1" V 3530 3700 50  0000 C CNN
-F 1 "47" V 3450 3700 50  0000 C CNN
+F 1 "33" V 3450 3700 50  0000 C CNN
 F 2 "Resistors_ThroughHole:Resistor_Horizontal_RM15mm" V 3380 3700 50  0001 C CNN
 F 3 "" H 3450 3700 50  0000 C CNN
@@
 	3900 3800 3900 3550
 $Comp
-L GND #PWR01
+L GND #PWR2
 U 1 1 5911CC63
 P 4000 4300
-F 0 "#PWR01" H 4000 4050 50  0001 C CNN
+F 0 "#PWR2" H 4000 4050 50  0001 C CNN
 F 1 "GND" H 4000 4150 50  0000 C CNN
 F 2 "" H 4000 4300 50  0000 C CNN
@@
 	1    4000 4300
 	1    0    0    -1
-$EndComp
-$Comp
-L Q_PNP_BCE Q2
-U 1 1 5911CEF1
-P 4200 4000
-F 0 "Q2" H 4100 3850 50  0000 L CNN
-F 1 "ASZ15" H 4000 4200 50  0000 L CNN
-F 2 "TO_SOT_Packages_THT:TO3" H 4400 4100 50  0001 C CNN
-F 3 "" H 4200 4000 50  0000 C CNN
-	1    4200 4000
-	-1   0    0    1
 $EndComp
 $Comp
@@
 F 3 "" H 4550 4000 50  0000 C CNN
 	1    4550 4000
-	-1   0    0    -1
+	1    0    0    1
 $EndComp
 $Comp
-L R R3
+L R R2
 U 1 1 5911CEFD
 P 4550 3700
-F 0 "R3" V 4630 3700 50  0000 C CNN
-F 1 "47" V 4550 3700 50  0000 C CNN
+F 0 "R2" V 4630 3700 50  0000 C CNN
+F 1 "33" V 4550 3700 50  0000 C CNN
 F 2 "Resistors_ThroughHole:Resistor_Horizontal_RM15mm" V 4480 3700 50  0001 C CNN
 F 3 "" H 4550 3700 50  0000 C CNN
@@
 	3500 4000 3600 4000
 $Comp
-L R R2
+L R R3
 U 1 1 5911D07F
 P 3550 4200
-F 0 "R2" V 3630 4200 50  0000 C CNN
+F 0 "R3" V 3630 4200 50  0000 C CNN
 F 1 "1k" V 3550 4200 50  0000 C CNN
 F 2 "Resistors_ThroughHole:Resistor_Horizontal_RM15mm" V 3480 4200 50  0001 C CNN
@@
 $EndComp
 $Comp
-L GND #PWR02
+L GND #PWR1
 U 1 1 5911D1E8
 P 3550 4850
-F 0 "#PWR02" H 3550 4600 50  0001 C CNN
+F 0 "#PWR1" H 3550 4600 50  0001 C CNN
 F 1 "GND" H 3550 4700 50  0000 C CNN
 F 2 "" H 3550 4850 50  0000 C CNN
@@
 	1    0    0    -1
 $EndComp
+$Comp
+L Q_NPN_BCE Q2
+U 1 1 5918EEC6
+P 4200 4000
+F 0 "Q2" H 4100 3850 50  0000 L CNN
+F 1 "KD503" H 4000 4200 50  0000 L CNN
+F 2 "" H 4400 4100 50  0000 C CNN
+F 3 "" H 4200 4000 50  0000 C CNN
+	1    4200 4000
+	-1   0    0    1
+$EndComp
+$Comp
+L Q_NPN_BCE Q1
+U 1 1 5918EF71
+P 3800 4000
+F 0 "Q1" H 3700 3850 50  0000 L CNN
+F 1 "KD503" H 3600 4200 50  0000 L CNN
+F 2 "" H 4000 4100 50  0000 C CNN
+F 3 "" H 3800 4000 50  0000 C CNN
+	1    3800 4000
+	1    0    0    1
+$EndComp
+Text Notes 3800 4850 0    60   ~ 0
+R1,R2: 15..100 ohm
 $EndSCHEMATC
