File: MOSFET-24V/pcb/kicad/royer.sch (KiCad schematic (older format))
At the start: 26 parts, among them J1 Screw_Terminal_1x04, Q1 IRFB4410, Q2 IRFD110, Q3 IRFD110, Q4 IRFB4410

Commit message: Cn 22nF comment
Parts:
- C1, C2, C3, C4: value 10nF -> 22nF
Other:
- note added: "Cn=10nF works. try Cn=22nF\nwith C1=C4=22nF C2=C3=10nF\nmosfets heat up and can lockup\non load.\nCn = 4*Cgs of output mosfet"
- note removed: "with C1=C4=22nF C2=C3=10nF\nmosfets heat up and can lockup\non load."
Changed lines of the file:
@@
 P 2550 4750
 F 0 "C1" H 2575 4850 50  0000 L CNN
-F 1 "10nF" H 2575 4650 50  0000 L CNN
+F 1 "22nF" H 2575 4650 50  0000 L CNN
 F 2 "Capacitors_SMD:C_1206_HandSoldering" H 2588 4600 50  0001 C CNN
 F 3 "" H 2550 4750 50  0000 C CNN
@@
 P 2750 4950
 F 0 "C2" H 2775 5050 50  0000 L CNN
-F 1 "10nF" H 2550 4850 50  0000 L CNN
+F 1 "22nF" H 2550 4850 50  0000 L CNN
 F 2 "Capacitors_SMD:C_1206_HandSoldering" H 2788 4800 50  0001 C CNN
 F 3 "" H 2750 4950 50  0000 C CNN
@@
 P 4250 4750
 F 0 "C4" H 4275 4850 50  0000 L CNN
-F 1 "10nF" H 4275 4650 50  0000 L CNN
+F 1 "22nF" H 4275 4650 50  0000 L CNN
 F 2 "Capacitors_SMD:C_1206_HandSoldering" H 4288 4600 50  0001 C CNN
 F 3 "" H 4250 4750 50  0000 C CNN
@@
 P 4050 4950
 F 0 "C3" H 4075 5050 50  0000 L CNN
-F 1 "10nF" H 3850 4850 50  0000 L CNN
+F 1 "22nF" H 3850 4850 50  0000 L CNN
 F 2 "Capacitors_SMD:C_1206_HandSoldering" H 4088 4800 50  0001 C CNN
 F 3 "" H 4050 4950 50  0000 C CNN
@@
 Text Label 6750 4700 0    60   ~ 0
 C2
-Text Notes 2650 7100 0    60   ~ 0
-with C1=C4=22nF C2=C3=10nF\nmosfets heat up and can lockup\non load.
+Text Notes 2650 7350 0    60   ~ 0
+Cn=10nF works. try Cn=22nF\nwith C1=C4=22nF C2=C3=10nF\nmosfets heat up and can lockup\non load.\nCn = 4*Cgs of output mosfet
 $EndSCHEMATC
